File: KiCad/TinyDivercityRX5808.kicad_pcb (KiCad board)
At the start: 2 copper layers, 37.4 x 23.7 mm, 23 parts, among them J1 Googles, SW1 SW_DPST, U1 MAX4624/5, U2 ATTINY85-20SU

Commit message: Initial writeup on firmware
Other:
- board text added: "100K"
- board text added: "100n"
- board text added: "10K"
- board text added: "10n"
- board text added: "10uf"
- board text added: "1K"
- board text added: "30"
- board text added: "AUDIO"
- board text added: "GND"
- board text added: "LED"
- board text added: "MISO"
- board text added: "MOSI"
- board text added: "RSSI"
- board text added: "RST"
- board text added: "S1"
- board text added: "S2"
- board text added: "S3"
- board text added: "SCK"
- board text added: "VCC"
- board text added: "VIDEO"
Changed lines of the file:
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@@
     (area 127.224999 90.374999 164.775001 114.225001)
     (thickness 1.6)
-    (drawings 8)
+    (drawings 56)
     (tracks 244)
     (zones 0)
@@
     )
   )
+  (gr_text VCC (at 164.1 97.45 90) (layer F.SilkS)
+    (effects (font (size 0.5 0.5) (thickness 0.1)))
+  )
+  (gr_text GND (at 164.1 99.95 90) (layer F.SilkS)
+    (effects (font (size 0.5 0.5) (thickness 0.1)))
+  )
+  (gr_text RST (at 158.1 102.55 90) (layer F.SilkS)
+    (effects (font (size 0.5 0.5) (thickness 0.1)))
+  )
+  (gr_text MOSI (at 158.1 97.35 90) (layer F.SilkS)
+    (effects (font (size 0.5 0.5) (thickness 0.1)))
+  )
+  (gr_text SCK (at 158.1 105.05 90) (layer F.SilkS)
+    (effects (font (size 0.5 0.5) (thickness 0.1)))
+  )
+  (gr_text MISO (at 158 107.65 90) (layer F.SilkS)
+    (effects (font (size 0.5 0.5) (thickness 0.1)))
+  )
+  (gr_text VCC (at 130.5 102.15 270) (layer F.SilkS)
+    (effects (font (size 0.5 0.5) (thickness 0.1)))
+  )
+  (gr_text AUDIO (at 130.5 97.25 270) (layer F.SilkS)
+    (effects (font (size 0.5 0.5) (thickness 0.1)))
+  )
+  (gr_text VIDEO (at 130.5 94.65 270) (layer F.SilkS)
+    (effects (font (size 0.5 0.5) (thickness 0.1)))
+  )
+  (gr_text GND (at 130.5 92.05 270) (layer F.SilkS)
+    (effects (font (size 0.5 0.5) (thickness 0.1)))
+  )
+  (gr_text GND (at 130.5 104.75 270) (layer F.SilkS)
+    (effects (font (size 0.5 0.5) (thickness 0.1)))
+  )
+  (gr_text S3 (at 130.5 107.25 270) (layer F.SilkS)
+    (effects (font (size 0.5 0.5) (thickness 0.1)))
+  )
+  (gr_text S2 (at 130.5 109.85 270) (layer F.SilkS)
+    (effects (font (size 0.5 0.5) (thickness 0.1)))
+  )
+  (gr_text S1 (at 130.5 112.35 270) (layer F.SilkS)
+    (effects (font (size 0.5 0.5) (thickness 0.1)))
+  )
+  (gr_text GND (at 133.2 93.75 180) (layer F.SilkS)
+    (effects (font (size 0.5 0.5) (thickness 0.1)))
+  )
+  (gr_text AUDIO (at 138.3 93.75 180) (layer F.SilkS)
+    (effects (font (size 0.5 0.5) (thickness 0.1)))
+  )
+  (gr_text VIDEO (at 135.7 93.75 180) (layer F.SilkS)
+    (effects (font (size 0.5 0.5) (thickness 0.1)))
+  )
+  (gr_text RSSI (at 140.8 93.75 180) (layer F.SilkS)
+    (effects (font (size 0.5 0.5) (thickness 0.1)))
+  )
+  (gr_text VCC (at 143.3 93.75 180) (layer F.SilkS)
+    (effects (font (size 0.5 0.5) (thickness 0.1)))
+  )
+  (gr_text GND (at 145.9 93.75 180) (layer F.SilkS)
+    (effects (font (size 0.5 0.5) (thickness 0.1)))
+  )
+  (gr_text S3 (at 148.4 93.75 180) (layer F.SilkS)
+    (effects (font (size 0.5 0.5) (thickness 0.1)))
+  )
+  (gr_text S2 (at 151 93.75 180) (layer F.SilkS)
+    (effects (font (size 0.5 0.5) (thickness 0.1)))
+  )
+  (gr_text S1 (at 153.5 93.75 180) (layer F.SilkS)
+    (effects (font (size 0.5 0.5) (thickness 0.1)))
+  )
+  (gr_text S1 (at 153.2 110.95) (layer F.SilkS)
+    (effects (font (size 0.5 0.5) (thickness 0.1)))
+  )
+  (gr_text S2 (at 150.6 110.95) (layer F.SilkS)
+    (effects (font (size 0.5 0.5) (thickness 0.1)))
+  )
+  (gr_text S3 (at 148.1 110.95) (layer F.SilkS)
+    (effects (font (size 0.5 0.5) (thickness 0.1)))
+  )
+  (gr_text VIDEO (at 135.4 110.95) (layer F.SilkS)
+    (effects (font (size 0.5 0.5) (thickness 0.1)))
+  )
+  (gr_text GND (at 132.9 110.95) (layer F.SilkS)
+    (effects (font (size 0.5 0.5) (thickness 0.1)))
+  )
+  (gr_text GND (at 145.5 110.95) (layer F.SilkS)
+    (effects (font (size 0.5 0.5) (thickness 0.1)))
+  )
+  (gr_text VCC (at 143 110.95) (layer F.SilkS)
+    (effects (font (size 0.5 0.5) (thickness 0.1)))
+  )
+  (gr_text RSSI (at 140.5 110.95) (layer F.SilkS)
+    (effects (font (size 0.5 0.5) (thickness 0.1)))
+  )
+  (gr_text 1K (at 134.1 110.25) (layer B.SilkS)
+    (effects (font (size 0.7 0.7) (thickness 0.15)) (justify mirror))
+  )
+  (gr_text 1K (at 134.1 108.85) (layer B.SilkS)
+    (effects (font (size 0.7 0.7) (thickness 0.15)) (justify mirror))
+  )
+  (gr_text 1K (at 134.1 107.35) (layer B.SilkS)
+    (effects (font (size 0.7 0.7) (thickness 0.15)) (justify mirror))
+  )
+  (gr_text LED (at 136.9 109.45) (layer F.SilkS)
+    (effects (font (size 0.7 0.7) (thickness 0.15)))
+  )
+  (gr_text LED (at 143.5 96.35) (layer F.SilkS)
+    (effects (font (size 0.7 0.7) (thickness 0.15)))
+  )
+  (gr_circle (center 142.3 106.45) (end 142.6 106.75) (layer F.SilkS) (width 0.2))
+  (gr_circle (center 135.3 103.65) (end 135.6 103.95) (layer F.SilkS) (width 0.2))
+  (gr_text 10uf (at 140.9 99.75) (layer F.SilkS)
+    (effects (font (size 0.7 0.7) (thickness 0.15)))
+  )
+  (gr_text 100n (at 141 103.75) (layer F.SilkS)
+    (effects (font (size 0.7 0.7) (thickness 0.15)))
+  )
+  (gr_text 100n (at 137.5 103.15) (layer F.SilkS)
+    (effects (font (size 0.7 0.7) (thickness 0.15)))
+  )
+  (gr_text 10n (at 137.6 99.05) (layer F.SilkS)
+    (effects (font (size 0.7 0.7) (thickness 0.15)))
+  )
+  (gr_text 10K (at 161.8 110.85) (layer F.SilkS)
+    (effects (font (size 0.7 0.7) (thickness 0.15)))
+  )
+  (gr_text 1K (at 147.6 95.85) (layer F.SilkS)
+    (effects (font (size 0.7 0.7) (thickness 0.15)))
+  )
+  (gr_text 100K (at 135.3 105.35) (layer F.SilkS)
+    (effects (font (size 0.7 0.7) (thickness 0.15)))
+  )
+  (gr_text 100K (at 140.7 97.85) (layer F.SilkS)
+    (effects (font (size 0.7 0.7) (thickness 0.15)))
+  )
+  (gr_text 30 (at 137 95.75) (layer F.SilkS)
+    (effects (font (size 0.7 0.7) (thickness 0.15)))
+  )
+  (gr_text 1K (at 137.2 107.95) (layer F.SilkS)
+    (effects (font (size 0.7 0.7) (thickness 0.15)))
+  )
   (dimension 23.7 (width 0.3) (layer Dwgs.User)

Commit message: Modified test board
Parts:
- added JP2: JVB, Pin_Headers:Pin_Header_Straight_1x02_Pitch2.54mm, F.Cu at (133.4, 108.5)
- added JP3: JWA, Pin_Headers:Pin_Header_Straight_1x02_Pitch2.54mm, F.Cu at (133.0, 95.5)
- moved R3 5.11 mm to (127.3, 112.3)
- moved R2 4.81 mm to (127.3, 109.8)
- moved J1 4.80 mm to (124.0, 112.3)
- moved R1 4.70 mm to (127.3, 107.2)
- moved SW1 0.30 mm to (153.3, 102.2)
Connections:
- U1 pad 4: /VideoA -> Net-(JP3-Pad2)
- U1 pad 6: /VideoB -> Net-(JP2-Pad2)
Routing:
- net VCC: track 63.7 -> 73.3 mm
- net Net-(JP2-Pad2): track 0.00 -> 7.49 mm
- net Net-(JP3-Pad2): track 0.00 -> 6.24 mm
- net /VideoB: track 11.0 -> 5.04 mm
- net Net-(J2-Pad3): track 40.9 -> 46.8 mm
- net Net-(J2-Pad1): track 43.5 -> 49.0 mm
- net Net-(J2-Pad2): track 42.2 -> 47.2 mm
- net /AUD_IN: track 7.48 -> 12.3 mm
- net /VideoA: track 9.74 -> 4.98 mm
- net GND: track 41.5 -> 45.7 mm
- net /VideoOut: track 10.2 -> 13.0 mm
- net /RST: track 27.9 -> 29.1 mm
- net Net-(J1-Pad1): track 3.61 -> 2.55 mm
Other:
- board size 37.4 x 23.7 mm -> 42.7 x 23.7 mm

Commit message: Second version of prototype board is ready
Parts:
- removed JP3: JWA, Pin_Headers:Pin_Header_Straight_1x02_Pitch2.54mm
- removed PROG: PROG, Pin_Headers:Pin_Header_Straight_2x05_Pitch2.54mm
- added C5: 100n, Capacitors_SMD:C_0603, F.Cu at (136.0, 104.1)
- added C6: 10n, Capacitors_SMD:C_0603, F.Cu at (137.6, 104.0)
- added D3: D_Schottky, Diodes_SMD:D_SOD-123, F.Cu at (158.8, 90.2)
- added J4: PROG, Pin_Headers:Pin_Header_Straight_2x05_Pitch2.54mm, F.Cu at (162.3, 97.5)
- added U3: MAX4625, TO_SOT_Packages_SMD:SOT-23-6, F.Cu at (132.7, 104.1)
- D1: footprint LEDs:LED_0603 -> LEDs:LED_0805
- D2: footprint LEDs:LED_0603 -> LEDs:LED_0805_HandSoldering
- JP2: value JVB -> Video4/5; footprint Pin_Headers:Pin_Header_Straight_1x02_Pitch2.54mm -> Pin_Headers:Pin_Header_Straight_1x03_Pitch2.54mm
- R6, R7, R8: footprint Resistors_SMD:R_0603 -> Resistors_SMD:R_1206
- U1: value MAX4624/5 -> MAX4624
- moved JP1 35.7 mm to (127.8, 108.4)
- moved R9 23.3 mm to (159.8, 87.6)
- moved D1 22.7 mm to (155.0, 93.0), turned to 90 degrees
- moved R6 18.3 mm to (156.1, 100.8), turned to 90 degrees
- moved D2 18.0 mm to (154.6, 109.4)
- moved R8 14.0 mm to (156.1, 105.8), turned to 270 degrees
- moved SW1 11.6 mm to (145.0, 94.1)
- moved JP2 10.5 mm to (123.8, 104.3), turned to 180 degrees
- moved C1 10.5 mm to (150.5, 99.5), turned to 180 degrees
- moved C4 9.64 mm to (150.5, 97.9), turned to 0 degrees
- moved R7 8.40 mm to (135.5, 88.8)
- moved RXA 6.72 mm to (153.3, 85.3)
- moved R4 6.47 mm to (141.6, 102.3), turned to 270 degrees
- moved U1 5.29 mm to (132.6, 96.6)
- moved J1 5.03 mm to (119.0, 112.5)
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Connections:
- C1 pad 1: Net-(C1-Pad1) -> /PROG_PWR
- C2 pad 1: Net-(C1-Pad1) -> /PROG_PWR
- C3 pad 2: Net-(C1-Pad1) -> /PROG_PWR
- C4 pad 2: Net-(C1-Pad1) -> /PROG_PWR
- J1 pad 6: Net-(J1-Pad6) -> /RSSI_G
- JP1 pad 1: VCC -> /RSSI_G
- JP1 pad 2: Net-(C1-Pad1) -> /RSSI_A
- JP2 pad 1: /VideoB -> Net-(JP2-Pad1)
- JP2 pad 2: Net-(JP2-Pad2) -> /VideoOut
- R6 pad 1: Net-(R6-Pad1) -> /SCK
- R9 pad 2: Net-(C1-Pad1) -> /PROG_PWR
- U1 pad 2: Net-(C1-Pad1) -> /PROG_PWR
- U1 pad 4: Net-(JP3-Pad2) -> /VideoA
- U1 pad 5: /VideoOut -> Net-(JP2-Pad3)
- U1 pad 6: Net-(JP2-Pad2) -> /VideoB
- U2 pad 2: Net-(R6-Pad1) -> /RSSI_A
- U2 pad 7: /RSSI_A -> /SCK
- U2 pad 8: Net-(C1-Pad1) -> /PROG_PWR
Routing:
- net GND: track 45.7 -> 177.6 mm, vias 5 -> 2
- net /PROG_PWR: track 0.00 -> 79.6 mm, vias 0 -> 3
- net Net-(C1-Pad1): track 56.6 -> 0.00 mm
- net /MOSI: track 33.6 -> 85.5 mm, vias 2 -> 1
- net VCC: track 73.3 -> 101.6 mm
- net /VideoA: track 4.98 -> 23.9 mm, vias 0 -> 2
- net /VideoB: track 5.04 -> 23.7 mm
- net Net-(J2-Pad1): track 49.0 -> 64.3 mm, vias 1 -> 0
- net Net-(J2-Pad2): track 47.2 -> 62.0 mm, vias 2 -> 0
- net /RSSI_G: track 0.00 -> 14.7 mm
- net Net-(J2-Pad3): track 46.8 -> 60.9 mm
- net /RSSI_A: track 27.9 -> 41.7 mm, vias 0 -> 1
- net /MISO: track 24.6 -> 11.9 mm
- net /SCK: track 0.00 -> 12.0 mm
- net Net-(R6-Pad1): track 9.22 -> 0.00 mm
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- removed copper zone on B.Cu, net GND
- removed copper zone on F.Cu, net GND
Other:
- board size 42.7 x 23.7 mm -> 52 x 34.5 mm
- net class Default: clearance 0.2 -> 0.3; trace_width 0.3 -> 0.5; via_dia 1.2 -> 1.5
- net class GND added: clearance 0.3, trace_width 0.6, via_dia 1.5, via_drill 0.5
- net class VCC: via_dia 1.2 -> 1.5
- rule trace_clearance: 0.2 -> 0.3

Commit message: Slight asjustment to the PCB
Parts:
- D2: footprint LEDs:LED_0805_HandSoldering -> LEDs:LED_0805
Changed lines of the file:
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@@
     (links 75)
     (no_connects 2)
-    (area 115.724999 82.474999 167.875001 117.125001)
+    (area 115.717619 82.474999 179.15 123.250001)
     (thickness 1.6)
-    (drawings 54)
+    (drawings 56)
     (tracks 335)
     (zones 0)
@@
   )
   (setup
-    (last_trace_width 0.3)
+    (last_trace_width 0.5)
     (user_trace_width 0.3)
     (trace_clearance 0.3)
@@
     )
   )
-  (module LEDs:LED_0805_HandSoldering (layer F.Cu)
-    (at 154.59 109.36 180)
-    (descr "Resistor SMD 0805, hand soldering")
-    (tags "resistor 0805")
-    (attr smd)
-    (fp_text reference D2 (at 0 -1.7 180) (layer F.SilkS) hide
-      (effects (font (size 1 1) (thickness 0.15)))
-    )
-    (fp_text value LED (at 0 1.75 180) (layer F.Fab) hide
-      (effects (font (size 1 1) (thickness 0.15)))
-    )
-    (fp_line (start -0.4 -0.4) (end -0.4 0.4) (layer F.Fab) (width 0.1))
-    (fp_line (start -0.4 0) (end 0.2 -0.4) (layer F.Fab) (width 0.1))
-    (fp_line (start 0.2 0.4) (end -0.4 0) (layer F.Fab) (width 0.1))
-    (fp_line (start 0.2 -0.4) (end 0.2 0.4) (layer F.Fab) (width 0.1))
-    (fp_line (start -1 0.62) (end -1 -0.62) (layer F.Fab) (width 0.1))
-    (fp_line (start 1 0.62) (end -1 0.62) (layer F.Fab) (width 0.1))
-    (fp_line (start 1 -0.62) (end 1 0.62) (layer F.Fab) (width 0.1))
-    (fp_line (start -1 -0.62) (end 1 -0.62) (layer F.Fab) (width 0.1))
-    (fp_line (start 1 0.75) (end -2.2 0.75) (layer F.SilkS) (width 0.12))
-    (fp_line (start -2.2 -0.75) (end 1 -0.75) (layer F.SilkS) (width 0.12))
-    (fp_line (start -2.35 -0.9) (end 2.35 -0.9) (layer F.CrtYd) (width 0.05))
-    (fp_line (start -2.35 -0.9) (end -2.35 0.9) (layer F.CrtYd) (width 0.05))
-    (fp_line (start 2.35 0.9) (end 2.35 -0.9) (layer F.CrtYd) (width 0.05))
-    (fp_line (start 2.35 0.9) (end -2.35 0.9) (layer F.CrtYd) (width 0.05))
-    (fp_line (start -2.2 -0.75) (end -2.2 0.75) (layer F.SilkS) (width 0.12))
-    (pad 1 smd rect (at -1.35 0 180) (size 1.5 1.3) (layers F.Cu F.Paste F.Mask)
-      (net 22 "Net-(D2-Pad1)"))
-    (pad 2 smd rect (at 1.35 0 180) (size 1.5 1.3) (layers F.Cu F.Paste F.Mask)
-      (net 2 VCC))
-    (model ${KISYS3DMOD}/LEDs.3dshapes/LED_0805.wrl
-      (at (xyz 0 0 0))
-      (scale (xyz 1 1 1))
-      (rotate (xyz 0 0 0))
-    )
-  )
   (module LEDs:LED_0805 (layer F.Cu)
     (at 155 92.98 90)
@@
       (effects (font (size 1 1) (thickness 0.15)))
     )
-    (fp_text value 30 (at 0 1.95) (layer F.Fab)
+    (fp_text value 30 (at 0 1.95) (layer F.Fab) hide
       (effects (font (size 1 1) (thickness 0.15)))
     )
@@
       (rotate (xyz 0 0 0))
     )
+  )
+  (module LEDs:LED_0805 (layer F.Cu)
+    (at 154.59 109.36 180)
+    (descr "LED 0805 smd package")
+    (tags "LED led 0805 SMD smd SMT smt smdled SMDLED smtled SMTLED")
+    (attr smd)
+    (fp_text reference D2 (at 0 -1.45 180) (layer F.SilkS) hide
+      (effects (font (size 1 1) (thickness 0.15)))
+    )
+    (fp_text value LED (at 0 1.55 180) (layer F.Fab)
+      (effects (font (size 1 1) (thickness 0.15)))
+    )
+    (fp_line (start -1.8 -0.7) (end -1.8 0.7) (layer F.SilkS) (width 0.12))
+    (fp_line (start -0.4 -0.4) (end -0.4 0.4) (layer F.Fab) (width 0.1))
+    (fp_line (start -0.4 0) (end 0.2 -0.4) (layer F.Fab) (width 0.1))
+    (fp_line (start 0.2 0.4) (end -0.4 0) (layer F.Fab) (width 0.1))
+    (fp_line (start 0.2 -0.4) (end 0.2 0.4) (layer F.Fab) (width 0.1))
+    (fp_line (start 1 0.6) (end -1 0.6) (layer F.Fab) (width 0.1))
+    (fp_line (start 1 -0.6) (end 1 0.6) (layer F.Fab) (width 0.1))
+    (fp_line (start -1 -0.6) (end 1 -0.6) (layer F.Fab) (width 0.1))
+    (fp_line (start -1 0.6) (end -1 -0.6) (layer F.Fab) (width 0.1))
+    (fp_line (start -1.8 0.7) (end 1 0.7) (layer F.SilkS) (width 0.12))
+    (fp_line (start -1.8 -0.7) (end 1 -0.7) (layer F.SilkS) (width 0.12))
+    (fp_line (start 1.95 -0.85) (end 1.95 0.85) (layer F.CrtYd) (width 0.05))
+    (fp_line (start 1.95 0.85) (end -1.95 0.85) (layer F.CrtYd) (width 0.05))
+    (fp_line (start -1.95 0.85) (end -1.95 -0.85) (layer F.CrtYd) (width 0.05))
+    (fp_line (start -1.95 -0.85) (end 1.95 -0.85) (layer F.CrtYd) (width 0.05))
+    (fp_text user %R (at 0 -1.25 180) (layer F.Fab)
+      (effects (font (size 0.4 0.4) (thickness 0.1)))
+    )
+    (pad 2 smd rect (at 1.1 0) (size 1.2 1.2) (layers F.Cu F.Paste F.Mask)
+      (net 2 VCC))
+    (pad 1 smd rect (at -1.1 0) (size 1.2 1.2) (layers F.Cu F.Paste F.Mask)
+      (net 22 "Net-(D2-Pad1)"))
+    (model ${KISYS3DMOD}/LEDs.3dshapes/LED_0805.wrl
+      (at (xyz 0 0 0))
+      (scale (xyz 1 1 1))
+      (rotate (xyz 0 0 180))
+    )
+  )
+  (dimension 52 (width 0.3) (layer Dwgs.User)
+    (gr_text "52,000 mm" (at 141.8 121.9) (layer Dwgs.User)
+      (effects (font (size 1.5 1.5) (thickness 0.3)))
+    )
+    (feature1 (pts (xy 115.8 117.05) (xy 115.8 123.25)))
+    (feature2 (pts (xy 167.8 117.05) (xy 167.8 123.25)))
+    (crossbar (pts (xy 167.8 120.55) (xy 115.8 120.55)))
+    (arrow1a (pts (xy 115.8 120.55) (xy 116.926504 119.963579)))
+    (arrow1b (pts (xy 115.8 120.55) (xy 116.926504 121.136421)))
+    (arrow2a (pts (xy 167.8 120.55) (xy 166.673496 119.963579)))
+    (arrow2b (pts (xy 167.8 120.55) (xy 166.673496 121.136421)))
+  )
+  (dimension 34.5 (width 0.3) (layer Dwgs.User)
+    (gr_text "34,500 mm" (at 172.65 99.8 270) (layer Dwgs.User)
+      (effects (font (size 1.5 1.5) (thickness 0.3)))
+    )
+    (feature1 (pts (xy 167.8 117.05) (xy 174 117.05)))
+    (feature2 (pts (xy 167.8 82.55) (xy 174 82.55)))
+    (crossbar (pts (xy 171.3 82.55) (xy 171.3 117.05)))
+    (arrow1a (pts (xy 171.3 117.05) (xy 170.713579 115.923496)))
+    (arrow1b (pts (xy 171.3 117.05) (xy 171.886421 115.923496)))
+    (arrow2a (pts (xy 171.3 82.55) (xy 170.713579 83.676504)))
+    (arrow2b (pts (xy 171.3 82.55) (xy 171.886421 83.676504)))
   )
   (gr_line (start 115.8 117.05) (end 115.8 116.55) (angle 90) (layer Edge.Cuts) (width 0.15))
@@
   (segment (start 133.66 95.67) (end 135.77 95.67) (width 0.6) (layer F.Cu) (net 1))
   (segment (start 135.77 95.67) (end 135.91 95.81) (width 0.6) (layer F.Cu) (net 1))
-  (segment (start 155 91.88) (end 156.7 90.18) (width 0.6) (layer F.Cu) (net 2) (status 400000))
-  (segment (start 156.7 90.18) (end 157.19 90.18) (width 0.6) (layer F.Cu) (net 2) (status 800000))
+  (segment (start 155 91.88) (end 156.7 90.18) (width 0.6) (layer F.Cu) (net 2))
+  (segment (start 156.7 90.18) (end 157.19 90.18) (width 0.6) (layer F.Cu) (net 2))
   (segment (start 143.17 85.79) (end 143.83 86.45) (width 0.6) (layer B.Cu) (net 2))
   (segment (start 143.84 105.99) (end 141.79 108.04) (width 0.6) (layer B.Cu) (net 2))
@@
   (segment (start 143.59 108.04) (end 152.075313 108.04) (width 0.6) (layer F.Cu) (net 2))
   (segment (start 143.59 108.04) (end 143.59 108.04) (width 0.6) (layer F.Cu) (net 2))
-  (segment (start 156.06 99.3) (end 155.96 99.2) (width 0.5) (layer F.Cu) (net 3) (status C00000))
-  (segment (start 155.96 99.2) (end 155.96 95.04) (width 0.5) (layer F.Cu) (net 3) (status 400000))
-  (segment (start 155.96 95.04) (end 155 94.08) (width 0.5) (layer F.Cu) (net 3) (status 800000))
+  (segment (start 156.06 99.3) (end 155.96 99.2) (width 0.5) (layer F.Cu) (net 3))
+  (segment (start 155.96 99.2) (end 155.96 95.04) (width 0.5) (layer F.Cu) (net 3))
+  (segment (start 155.96 95.04) (end 155 94.08) (width 0.5) (layer F.Cu) (net 3))
   (segment (start 156.1 99.45) (end 156.06 99.49) (width 0.5) (layer F.Cu) (net 3) (status 30))
   (segment (start 118.97 112.46) (end 121.52 112.46) (width 0.5) (layer B.Cu) (net 4))

Commit message: First draft of final PCB
Parts:
- removed C5: 100n, Capacitors_SMD:C_0603
- removed C6: 10n, Capacitors_SMD:C_0603
- removed JP1: Jumper, Pin_Headers:Pin_Header_Straight_1x02_Pitch2.54mm
- removed JP2: Video4/5, Pin_Headers:Pin_Header_Straight_1x03_Pitch2.54mm
- removed RXA: RX_A, Pin_Headers:Pin_Header_Straight_1x09_Pitch2.54mm
- removed RXB: RX_B, Pin_Headers:Pin_Header_Straight_1x09_Pitch2.54mm
- removed U3: MAX4625, TO_SOT_Packages_SMD:SOT-23-6
- added J2: RX_A, KiCadCustomLibs:Pads_9pin_chess, F.Cu at (130.3, 99.7)
- added J3: RX_B, KiCadCustomLibs:Pads_9pin_chess, F.Cu at (147.1, 99.9)
- D1, D2: footprint LEDs:LED_0805 -> LEDs:LED_0402
- D3: footprint Diodes_SMD:D_SOD-123 -> Diodes_SMD:D_SOD-523
- J1: footprint Pin_Headers:Pin_Header_Straight_1x09_Pitch2.54mm -> Connectors_Molex:Molex_PicoBlade_53047-0910_09x1.25mm_Straight
- J4: value PROG -> Conn_01x06; footprint Pin_Headers:Pin_Header_Straight_2x05_Pitch2.54mm -> KiCadCustomLibs:Pads_prog_6pin1.25mm; moved to B.Cu
- R4, R5, R9: moved to B.Cu
- R6: footprint Resistors_SMD:R_1206 -> Resistors_SMD:R_0603; moved to B.Cu
- R7: value 30 -> 1K; footprint Resistors_SMD:R_1206 -> Resistors_SMD:R_0603; moved to B.Cu
- R8: value 1K -> 30; footprint Resistors_SMD:R_1206 -> Resistors_SMD:R_0603; moved to B.Cu
- SW1: value SW_DPST -> SW_Push; footprint Buttons_Switches_SMD:SW_SPST_B3S-1000 -> KiCadCustomLibs:Button_TS-018
- U2: value ATTINY85-20SU -> ATTINY85-20MU; footprint Housings_SOIC:SO-8_5.3x6.2mm_Pitch1.27mm -> Housings_DFN_QFN:QFN-20-1EP_4x4mm_Pitch0.5mm
- moved J1 26.1 mm to (144.8, 108.5)
- moved R8 24.2 mm to (132.3, 101.4), turned to 90 degrees
- moved D2 24.0 mm to (136.6, 93.5), turned to 90 degrees
- moved R3 23.0 mm to (145.2, 110.6), turned to 270 degrees
- moved J4 22.0 mm to (140.6, 93.6), turned to 180 degrees
- moved R9 21.8 mm to (139.7, 96.1), turned to 270 degrees
- moved R2 21.3 mm to (143.6, 110.6), turned to 270 degrees
- moved R1 19.9 mm to (141.9, 110.6), turned to 270 degrees
- moved C1 15.3 mm to (135.3, 101.7)
- moved R6 14.4 mm to (142.4, 96.2), turned to 0 degrees
- moved D3 13.1 mm to (146.2, 93.7), turned to 0 degrees
- moved SW1 13.1 mm to (132.0, 93.0), turned to 0 degrees
- moved D1 11.9 mm to (143.2, 93.5)
- moved C4 10.6 mm to (139.9, 98.2), turned to 180 degrees
- moved U1 8.39 mm to (135.3, 104.5), turned to 270 degrees
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Connections:
- J1 pad 6: /RSSI_G -> /RSSI_A
- J4 pad 1: /MOSI -> /PROG_PWR
- J4 pad 2: /PROG_PWR -> /MOSI
- J4 pad 3: Net-(J4-Pad3) -> GND
- J4 pad 4: GND -> /RST
- J4 pad 5: /RST -> /SCK
- J4 pad 6: GND -> /MISO
- R7 pad 1: /AUD_IN -> /MISO
- R7 pad 2: /AUD_OUT -> Net-(D2-Pad1)
- R8 pad 1: /MISO -> /AUD_IN
- R8 pad 2: Net-(D2-Pad1) -> /AUD_OUT
- U1 pad 5: Net-(JP2-Pad3) -> /VideoOut
- U2 pad 3: /RSSI_B -> (no net)
- U2 pad 4: GND -> (no net)
- U2 pad 5: /MOSI -> /RSSI_B
- U2 pad 6: /MISO -> (no net)
- U2 pad 7: /SCK -> (no net)
- U2 pad 8: /PROG_PWR -> GND
Routing:
- net GND: track 177.6 -> 6.99 mm, vias 2 -> 0
- net /MOSI: track 85.5 -> 20.6 mm, vias 1 -> 2
- net /PROG_PWR: track 79.6 -> 23.8 mm, vias 3 -> 2
- net VCC: track 101.6 -> 60.8 mm, vias 1 -> 3
- net /RSSI_A: track 41.7 -> 18.8 mm, vias 1 -> 2
- net Net-(J2-Pad1): track 64.3 -> 44.2 mm, vias 0 -> 3
- net Net-(J2-Pad3): track 60.9 -> 42.8 mm, vias 0 -> 2
- net Net-(J2-Pad2): track 62.0 -> 45.4 mm, vias 0 -> 3
- net /RSSI_G: track 14.7 -> 0.00 mm
- net /VideoA: track 23.9 -> 11.3 mm
- net /RST: track 34.2 -> 22.2 mm, vias 1 -> 3
- net /VideoB: track 23.7 -> 12.4 mm, vias 0 -> 2
- net Net-(JP2-Pad3): track 8.92 -> 0.00 mm
- net Net-(JP2-Pad1): track 8.84 -> 0.00 mm, vias 1 -> 0
- net /AUD_IN: track 20.5 -> 12.3 mm, vias 0 -> 1
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Other:
- board size 52 x 34.5 mm -> 22 x 20 mm
- net class Default: clearance 0.3 -> 0.1524; trace_width 0.5 -> 0.1524; via_dia 1.5 -> 0.6; via_drill 0.5 -> 0.254
- net class GND: clearance 0.3 -> 0.2; trace_width 0.6 -> 0.3; via_dia 1.5 -> 1; via_drill 0.5 -> 0.4
- net class VCC: clearance 0.3 -> 0.1524; trace_width 0.6 -> 0.3; via_dia 1.5 -> 1; via_drill 0.5 -> 0.4
- rule pad_to_mask_clearance: 0.15 -> 0.06
- rule trace_clearance: 0.3 -> 0.1524
- rule trace_min: 0.2 -> 0.1524
- rule via_min_drill: 0.3 -> 0.254
- board text added: "A"
- board text added: "B"
- board text added: "PROG"
- board text removed: "100K"
- board text removed: "100n"
- board text removed: "10K"
- board text removed: "10n"
- board text removed: "10uf"
- board text removed: "1K"
- board text removed: "30"
- board text removed: "AUDIO"
- board text removed: "GND"
- board text removed: "LED"
- board text removed: "MISO"
- board text removed: "MOSI"
- board text removed: "RSSI"
- board text removed: "RST"
- board text removed: "S1"
- board text removed: "S2"
- board text removed: "S3"
- board text removed: "SCK"
- board text removed: "VCC"
- board text removed: "VIDEO"
